File: revlp/41_1353/41_1353_pcb/r41l2.kicad_pcb (KiCad board)
At the start: 2 copper layers, 29.6 x 19.9 mm, 87 parts, among them SW01 SW_SPDT, SW02 SW_Push, U1 ProMicro

Commit message: [keyboard] reviung41_1353: Initial release
Parts:
- removed BT01: Battery_Cell, keeblib:cell_pads
- removed SW02: SW_Push, keeblib:alps_sksn
- added G***: LOGO, keeblib:chain_200mm, B.Cu at (133.0, 0.03)
- added REF**: OSHW-Symbol_13.4x12mm_SilkScreen, Symbol:OSHW-Symbol_13.4x12mm_SilkScreen, B.Cu at (145.8, 24.8)
- added REF**: edgecuts_r41l2_pcb, 41_1353:edgecuts_r41l2_pcb, F.Cu at (146.0, -10.4)
- SW01: moved to B.Cu
- SwG2: footprint keeblib:pg1353_reversible_2u -> keeblib:pg1353_2u
- U1: footprint keeblib:ArduinoProMicro -> keebMCU:ProMicroNiced
- moved D_E2 189.3 mm to (196.5, 14.6), turned to 193 degrees
- moved D_D1 186.1 mm to (174.7, 4.64), turned to 193 degrees
- moved SwE2 185.2 mm to (197.7, 19.5), turned to 13 degrees
- moved SwD1 182.3 mm to (175.9, 9.52), turned to 13 degrees
- moved D_E0 171.2 mm to (161.5, 31.7), turned to 193 degrees
- moved SwE0 168.6 mm to (162.6, 36.6), turned to 13 degrees
- moved SwD0 166.2 mm to (158.3, 18.1), turned to 13 degrees
- moved D_D0 165.2 mm to (157.2, 13.2), turned to 193 degrees
- moved D_F0 163.6 mm to (165.8, 50.2), turned to 193 degrees
- moved D_E1 162.4 mm to (179.0, 23.2), turned to 193 degrees
- moved SwF0 158.8 mm to (166.9, 55.1), turned to 13 degrees
- moved SwE1 158.1 mm to (180.1, 28.0), turned to 13 degrees
- moved D_E3 155.2 mm to (216.0, 14.6), turned to 193 degrees
- moved SwE3 151.6 mm to (217.2, 19.5), turned to 13 degrees
- moved D_E4 124.9 mm to (235.5, 14.6), turned to 193 degrees
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Connections:
- SW01 pad 1: Net-(BT01-Pad2) -> Net-(SW01-Pad1)
- U1 pad 22: RST -> (no net)
- U1 pad 24: RAW -> Net-(U1-Pad24)
Routing:
- net col4: track 92.8 -> 281.6 mm, vias 0 -> 1
- net col3: track 103.5 -> 277.9 mm, vias 0 -> 1
- net col2: track 122.7 -> 295.2 mm, vias 0 -> 2
- net col0: track 160.1 -> 332.0 mm, vias 0 -> 1
- net rowG: track 23.6 -> 190.0 mm
- net rowF: track 0.00 -> 164.0 mm, vias 0 -> 1
- net col1: track 141.8 -> 304.7 mm, vias 0 -> 2
- net rowE: track 0.00 -> 147.6 mm, vias 0 -> 1
- net col5: track 75.9 -> 221.5 mm
- net rowD: track 0.00 -> 129.9 mm, vias 0 -> 1
- net GND: track 0.00 -> 22.8 mm
- net rowA: track 113.9 -> 133.5 mm
- net Net-(D_D0-Pad2): track 0.00 -> 10.7 mm
- net Net-(D_G3-Pad2): track 0.00 -> 10.7 mm
- net Net-(D_F0-Pad2): track 0.00 -> 10.7 mm
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Other:
- board size 29.6 x 19.9 mm -> 251.3 x 103.7 mm
- board text added: "2021/06"
- board text added: "Concept :: Reviung41_1353"
- board text added: "github.com/cyril279/keyboards"
