File: revlp/41_1353/41_1353_pcb/r41l2.kicad_pcb (KiCad board)
At the start: 2 copper layers, 29.6 x 19.9 mm, 87 parts, among them SW01 SW_SPDT, SW02 SW_Push, U1 ProMicro

Commit message: r41l2: pcb development
Parts:
- removed BT01: Battery_Cell, keeblib:cell_pads
- removed SW02: SW_Push, keeblib:alps_sksn
- SW01: moved to B.Cu
- SwG2: footprint keeblib:pg1353_reversible_2u -> keeblib:pg1353_2u
- U1: footprint keeblib:ArduinoProMicro -> keebMCU:ProMicroNiced
- moved D_E2 197.3 mm to (186.8, 21.4), turned to 206 degrees
- moved D_D1 194.8 mm to (163.3, 16.6), turned to 206 degrees
- moved SwE2 192.3 mm to (189.0, 25.9)
- moved SwD1 190.0 mm to (165.5, 21.1)
- moved D_E1 172.1 mm to (171.7, 33.7), turned to 206 degrees
- moved D_E0 172.0 mm to (156.5, 46.0), turned to 206 degrees
- moved SwD0 169.7 mm to (150.4, 33.4)
- moved D_D0 169.6 mm to (148.2, 28.9), turned to 206 degrees
- moved D_F0 169.3 mm to (164.8, 63.0), turned to 206 degrees
- moved SwE0 168.5 mm to (158.7, 50.5)
- moved SwE1 166.9 mm to (173.8, 38.2)
- moved D_E3 164.1 mm to (205.8, 17.0), turned to 206 degrees
- moved SwF0 163.4 mm to (167.0, 67.5)
- moved SwE3 159.5 mm to (208.0, 21.5)
- moved D_E4 135.3 mm to (224.8, 12.7), turned to 206 degrees
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Connections:
- SW01 pad 1: Net-(BT01-Pad2) -> Net-(SW01-Pad1)
- U1 pad 22: RST -> (no net)
- U1 pad 24: RAW -> Net-(U1-Pad24)
Routing:
- net col0: track 160.1 -> 332.9 mm, vias 0 -> 1
- net col2: track 122.7 -> 294.0 mm, vias 0 -> 2
- net rowG: track 23.6 -> 191.7 mm
- net rowF: track 0.00 -> 164.0 mm, vias 0 -> 1
- net col1: track 141.8 -> 303.1 mm, vias 0 -> 2
- net rowE: track 0.00 -> 147.5 mm, vias 0 -> 1
- net col5: track 75.9 -> 220.6 mm
- net rowD: track 0.00 -> 129.5 mm, vias 0 -> 1
- net col4: track 92.8 -> 221.3 mm, vias 0 -> 1
- net col3: track 103.5 -> 214.2 mm, vias 0 -> 1
- net GND: track 0.00 -> 22.8 mm
- net rowA: track 113.9 -> 135.9 mm
- net Net-(D_D0-Pad2): track 0.00 -> 10.7 mm
- net Net-(D_G3-Pad2): track 0.00 -> 10.7 mm
- net Net-(D_F0-Pad2): track 0.00 -> 10.7 mm
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