File: one42/one42_pcb/one42_matrix.kicad_sch (KiCad schematic)
At the start: 84 parts

Commit message: [one42] version 1.0
- Relocated corner-thumb switch diodes
- Removed encoder base-supply option
- Fixed 'R5' silkscreen
- Fixed programmer-header V+ to 3v3
- Moved power sw. inboard
- Mounting holes routed to ground
- Battery-pad size reduced
- Relocated power-routing/switching components
- Repositioned 'XLII' text
Connections:
- net COL06: now also SwD06.1; no longer SwD06.2
- net COL07: now also SwD07.1; no longer SwD07.2
- net at D40.2 (A): now also SwD06.2; no longer SwD06.1
- net at D41.2 (A): now also SwD07.2; no longer SwD07.1
Changed lines of the file:
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@@
     (pin "2")
   )
-  (symbol (lib_id "Switch:SW_Push") (at 162.56 120.65 0) (unit 1)
+  (symbol (lib_name "SW_Push_2") (lib_id "Switch:SW_Push") (at 162.56 120.65 0) (mirror y) (unit 1)
     (in_bom yes) (on_board yes)
     (property "Reference" "SwD06" (id 0) (at 162.56 113.411 0))
@@
     (pin "2")
   )
-  (symbol (lib_id "Switch:SW_Push") (at 179.07 120.65 0) (unit 1)
+  (symbol (lib_name "SW_Push_1") (lib_id "Switch:SW_Push") (at 179.07 120.65 0) (mirror y) (unit 1)
     (in_bom yes) (on_board yes)
     (property "Reference" "SwD07" (id 0) (at 179.07 113.411 0))
