File: one42/one42_pcb/one42.kicad_pcb (KiCad board)
At the start: 2 copper layers, 252.3 x 111.8 mm, 121 parts, among them J1 Conn_01x04_Female, Q1 AO3401A, SW44 SW_SPDT, U1 TP4054, U2 AP2112K-3.3, U3 nRF52840_holyiot_18010, U4 One42

Commit message: [one42] version 1.0
- Relocated corner-thumb switch diodes
- Removed encoder base-supply option
- Fixed 'R5' silkscreen
- Fixed programmer-header V+ to 3v3
- Moved power sw. inboard
- Mounting holes routed to ground
- Battery-pad size reduced
- Relocated power-routing/switching components
- Repositioned 'XLII' text
Parts:
- removed H1, H2, H3, H4, H5, H6, H7, H8: MountingHole, MountingHole:MountingHole_2.2mm_M2_Pad
- removed JP1: EncoderPolarity, Jumper:SolderJumper-3_P1.3mm_Open_RoundedPad1.0x1.5mm
- moved D42 51.5 mm to (126.9, 88.6), turned to -90 degrees
- moved U1 46.2 mm to (97.2, 89.0), turned to -165 degrees
- moved R4 45.5 mm to (92.8, 91.0), turned to -165 degrees
- moved R2 44.8 mm to (67.9, 49.9), turned to 0 degrees
- moved R5 41.8 mm to (80.6, 31.1)
- moved SwC05 41.8 mm to (47.5, 78.9)
- moved SwC11 41.8 mm to (185.1, 59.5)
- moved SwD04 41.8 mm to (40.9, 97.7)
- moved D32 41.8 mm to (108.6, 64.4)
- moved SwA05 41.8 mm to (57.2, 42.6)
- moved F1 41.8 mm to (77.6, 31.6)
- moved D1 41.8 mm to (-33.6, 18.4)
- moved D12 41.8 mm to (174.1, 18.3)
- moved D15 41.8 mm to (0.49, 36.5)
- moved D36 41.8 mm to (183.8, 54.6)
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Connections:
- net /PVIN renamed /VSRC
- net Net-(BT1-Pad2) renamed /BattSw
- J1 pad 1: VBUS -> VDD_NRF
- SwD03 pad C: /encBASE -> GND
- SwD08 pad C: /encBASE -> GND
Routing:
- net /encBASE: track 113.5 -> 0.00 mm, vias 1 -> 0
- net VBUS: track 129.9 -> 90.9 mm, vias 3 -> 2
- net VDD_NRF: track 11.9 -> 47.6 mm, vias 0 -> 2
- net Net-(D37-Pad2): track 19.4 -> 9.11 mm
- net VBAT: track 82.4 -> 90.5 mm
- net ROWD: track 195.5 -> 203.4 mm
- net /charge: track 59.6 -> 66.3 mm
- net /BattSw: track 93.1 -> 98.5 mm
- net SWC: track 30.0 -> 25.7 mm, vias 1 -> 0
- net SWD: track 31.1 -> 27.4 mm, vias 1 -> 0
- net ROWA: track 321.6 -> 318.1 mm
- net Net-(D46-Pad1): track 10.7 -> 7.31 mm
- net COL06: track 90.1 -> 86.9 mm
- net VTAP: track 29.4 -> 26.4 mm
- net Net-(D45-Pad1): track 8.12 -> 5.23 mm
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Other:
- board text added: "+3v3"

Commit message: [one42] Version 1.0: Component-layout tweaks
- Moved power sw. to left-side of USB
- Moved LED's both to right-side of USB
Parts:
- moved JP3 27.0 mm to (56.7, 30.2)
- moved R7 26.7 mm to (83.5, 30.4)
- moved SW44 23.8 mm to (59.1, 23.8), turned to 174 degrees
- moved D46 17.2 mm to (80.3, 25.8), turned to -90 degrees
- turned C1 to 0 degrees
- turned D45 to -90 degrees
Routing:
- net /BattSw: track 98.5 -> 90.0 mm
- net RESET: track 45.9 -> 38.5 mm
- net VBUS: track 90.9 -> 88.8 mm
- net Net-(D45-Pad1): track 5.23 -> 6.65 mm
- net /VSRC: track 13.3 -> 14.6 mm
- net Net-(D46-Pad1): track 7.31 -> 6.08 mm
- net VTAP: track 26.4 -> 25.1 mm
- net ROWB: track 291.5 -> 290.3 mm
- net LED_1: track 50.7 -> 49.8 mm, vias 2 -> 3
- net VBAT: track 90.5 -> 91.4 mm
- net GND: track 8.27 -> 8.10 mm, vias 17 -> 12

Commit message: [one42] Version 1.0: Cleanup
Parts:
- moved R6 0.90 mm to (60.3, 31.4)
- moved C4 0.90 mm to (63.3, 31.9)
- moved R1 0.90 mm to (74.3, 33.4), turned to -90 degrees
- moved R3 0.90 mm to (66.3, 33.4)
- moved SW44 0.76 mm to (59.8, 24.1), turned to 175 degrees
- moved JP3 0.53 mm to (57.0, 30.6)
- moved R7 0.49 mm to (83.0, 30.6)
- moved R5 0.46 mm to (80.3, 31.4)
- moved F1 0.46 mm to (77.3, 31.9)
- moved D46 0.25 mm to (80.0, 25.9)
- moved D45 0.21 mm to (77.3, 25.9)
Routing:
- net GND: track 8.10 -> 5.14 mm, vias 12 -> 10
- net ROWA: track 318.2 -> 317.2 mm
- net /SHIELD: track 25.0 -> 24.5 mm
- net RESET: track 38.5 -> 37.9 mm
- net Net-(D7-Pad2): track 12.7 -> 13.3 mm
- net LED_1: track 49.8 -> 49.4 mm, vias 3 -> 4
Other:
- rule pad_to_mask_clearance: 0.051 -> 0
- board text removed: "+3v3"
- board text removed: "+V"
- board text removed: "GND"
- board text removed: "SWC"
- board text removed: "SWD"
